File: Lamply.sch (KiCad schematic (older format))
At the start: 51 parts, among them P1 CONN_01X04, P2 CONN_01X04, P3 CONN_01X04, P4 CONN_01X04, P5 CONN_02X10, P7 CONN_01X04, P8 CONN_01X04, SW1 SETUP, SW2 RESET, U1 PAM2305, U2 P1

Commit message: Simon overhaul assist
Parts:
- removed P5: CONN_02X10, particle:CONN-20-BIG, symbol CONN_02X10
- removed W4, W6: TEST_1P, Measurement_Points:Measurement_Point_Square-SMD-Pad_Small, symbol TEST_1P
- added JP1: JUMPER, Oddities:NetTie-I, symbol JUMPER
- added W13: TCK, Measurement_Points:Measurement_Point_Square-SMD-Pad_Small, symbol TEST_1P
- added W16: TRST, Measurement_Points:Measurement_Point_Square-SMD-Pad_Small, symbol TEST_1P
- added W17: gND, Measurement_Points:Measurement_Point_Square-SMD-Pad_Small, symbol TEST_1P
- added W8: 3V3, Measurement_Points:Measurement_Point_Square-SMD-Pad_Small, symbol TEST_1P
- W11: value TEST_1P -> JTAG_RST
- W12: value TEST_1P -> TDO
- W14: value TEST_1P -> TMS
- W15: value TEST_1P -> TDI
Connections:
- net +3V3: now also W8.1
- net A0: no longer W12.1
- net D0: now also R4.1, W3.1; no longer R1.2
- net D2: now also R1.2; no longer R4.1, W3.1
- net GND: now also P1.1 (P1), P2.1 (P1), P3.1 (P1), P4.1 (P1), P7.1 (P1), JP1.1; no longer C1.2, C10.2, C11.2, C2.2, C3.2, C4.2, C5.2, C6.2, C7.2, C8.2, C9.2, D3.1 (K), P1.4 (P4), P2.4 (P4), P3.4 (P4), P4.4 (P4), P7.4 (P4), U1.2 (GND), U2.1 (GND), U2.13 (GND), U2.15 (GND), U2.25 (GND), U2.28 (GND), U2.37 (GND), U2.39 (GND), U2.4 (GND), U2.59 (GND), U2.6 (GND), U2.65 (GND), U2.66 (GND), U2.67 (GND), U2.68 (GND), U2.69 (GND), U2.70 (GND), U2.71 (GND), U2.72 (GND), U2.73 (GND)
- net JTAG_RST: now also W11.1
- net TCK: now also W13.1
- net TDI: now also W15.1
- net TDO: now also W12.1
- net TMS: now also W14.1
- net TRST: now also W16.1
- net UVCC: now also P1.2 (P2), P2.2 (P2), P3.2 (P2), P4.2 (P2), P7.2 (P2); no longer P1.1 (P1), P2.1 (P1), P3.1 (P1), P4.1 (P1), P7.1 (P1)
- net at R1.1: now also P1.4 (P4); no longer P1.2 (P2)
- net at P1.3 (P3), R2.2: now also P2.4 (P4); no longer P2.2 (P2)
- net at P2.3 (P3), R4.2: now also P3.4 (P4); no longer P3.2 (P2)
- net at P3.3 (P3), R5.2: now also P4.4 (P4); no longer P4.2 (P2)
- net at P4.3 (P3), R6.2: now also P7.4 (P4); no longer P7.2 (P2)
- net at D2.3 (G), R8.2: no longer W14.1
- net at D2.4 (B), R7.2: no longer W11.1
- net at D2.2 (R), R9.2: no longer W15.1
- new net GNDA: C1.2, C10.2, C11.2, C2.2, C3.2, C4.2, C5.2, C6.2, C7.2, C8.2, C9.2, D3.1 (K), JP1.2, U1.2 (GND), U2.1 (GND), U2.13 (GND), U2.15 (GND), U2.25 (GND), U2.28 (GND), U2.37 (GND), U2.39 (GND), U2.4 (GND), U2.59 (GND), U2.6 (GND), U2.65 (GND), U2.66 (GND), U2.67 (GND), U2.68 (GND), U2.69 (GND), U2.70 (GND), U2.71 (GND), U2.72 (GND), U2.73 (GND), W17.1
- no-connect marks 27 -> 24
Other:
- note added: "Jumpers"
- moved on the sheet: R1
